File: ESP_uno.kicad_pcb (KiCad board)
At the start: 2 copper layers, 53.8 x 68.8 mm, 58 parts, among them J1 USB_C_Receptacle_USB2.0_14P, J2 Barrel, J3 Conn_01x08, J4 Conn_01x10, J5 Conn_01x06, J6 Conn_01x08, SW1 SW_MEC_5G, SW2 SW_MEC_5G, U1 ESP32-C3, U2 PAM2305AAB330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

Commit message: values
Parts:
- C1, C2, C3, C4: value C -> TBD
- C11, C5: value C -> 100nF
- R1, R2, R3, R4, R5: value R -> 5,1k
Changed lines of the file:
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@@
 			)
 		)
-		(property "Value" "R"
+		(property "Value" "5,1k"
 			(at 0 1.17 0)
 			(layer "F.Fab")
@@
 			)
 		)
-		(property "Value" "R"
+		(property "Value" "5,1k"
 			(at 0 1.17 0)
 			(layer "F.Fab")
@@
 			)
 		)
-		(property "Value" "R"
+		(property "Value" "5,1k"
 			(at 0 1.17 0)
 			(layer "F.Fab")
@@
 			)
 		)
-		(property "Value" "R"
+		(property "Value" "5,1k"
 			(at 0 1.17 90)
 			(layer "F.Fab")
@@
 			)
 		)
-		(property "Value" "C"
+		(property "Value" "100nF"
 			(at 0 1.16 90)
 			(layer "F.Fab")
@@
 			)
 		)
-		(property "Value" "C"
+		(property "Value" "TBD"
 			(at 0 1.16 90)
 			(layer "F.Fab")
@@
 			(net 48 "unconnected-(U2-FB-Pad4)")
 			(pinfunction "FB")
-			(pintype "input")
+			(pintype "input+no_connect")
 		)
 		(pad "5" smd roundrect
@@
 			)
 		)
-		(property "Value" "C"
+		(property "Value" "TBD"
 			(at 0 1.16 0)
 			(layer "F.Fab")
@@
 			)
 		)
-		(property "Value" "C"
+		(property "Value" "TBD"
 			(at 0 1.16 0)
 			(layer "F.Fab")
@@
 			)
 		)
-		(property "Value" "R"
+		(property "Value" "5,1k"
 			(at 0 1.17 90)
 			(layer "F.Fab")
@@
 			)
 		)
-		(property "Value" "C"
+		(property "Value" "100nF"
 			(at 0 1.16 90)
 			(layer "F.Fab")
@@
 			)
 		)
-		(property "Value" "C"
+		(property "Value" "TBD"
 			(at 0 1.16 90)
 			(layer "F.Fab")
