File: ESP_uno.kicad_sch (KiCad schematic)
At the start: 54 parts, among them J1 USB_C_Receptacle_USB2.0_14P, J2 Barrel, J3 Conn_01x08, J4 Conn_01x10, J5 Conn_01x06, J6 Conn_01x08, SW1 SW_MEC_5G, SW2 SW_MEC_5G, U1 ESP32-C3, U2 PAM2305AAB330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

Commit message: values
Parts:
- C1, C2, C3, C4: value C -> TBD
- C11, C5: value C -> 100nF
- R1, R2, R3, R4, R5: value R -> 5,1k
Connections:
- no-connect marks 8 -> 9
Changed lines of the file:
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@@
 	)
 	(no_connect
+		(at 87.63 60.96)
+	)
+	(no_connect
 		(at 167.64 78.74)
 	)
@@
 			)
 		)
-		(property "Value" "C"
+		(property "Value" "TBD"
 			(at 93.98 60.9662 0)
 			(effects
@@
 			)
 		)
-		(property "Value" "R"
+		(property "Value" "5,1k"
 			(at 54.61 59.69 90)
 			(effects
@@
 			)
 		)
-		(property "Value" "C"
+		(property "Value" "100nF"
 			(at 140.97 34.2962 0)
 			(effects
@@
 			)
 		)
-		(property "Value" "C"
+		(property "Value" "TBD"
 			(at 115.57 87.6362 0)
 			(effects
@@
 			)
 		)
-		(property "Value" "R"
+		(property "Value" "5,1k"
 			(at 56.134 68.072 90)
 			(effects
@@
 			)
 		)
-		(property "Value" "R"
+		(property "Value" "5,1k"
 			(at 29.21 101.6 0)
 			(effects
@@
 			)
 		)
-		(property "Value" "C"
+		(property "Value" "100nF"
 			(at 19.05 104.1462 0)
 			(effects
@@
 			)
 		)
-		(property "Value" "C"
+		(property "Value" "TBD"
 			(at 59.69 60.9662 0)
 			(effects
@@
 			)
 		)
-		(property "Value" "R"
+		(property "Value" "5,1k"
 			(at 134.874 34.29 90)
 			(effects
@@
 			)
 		)
-		(property "Value" "R"
+		(property "Value" "5,1k"
 			(at 175.26 50.8 0)
 			(effects
@@
 			)
 		)
-		(property "Value" "C"
+		(property "Value" "TBD"
 			(at 118.11 100.3362 0)
 			(effects
